Commit message: Swapped out camera mount to be accurate

File: src/authoring/urdfs/panda.urdf (robot description, URDF)
Before this commit: robot panda_kinect, 16 links, 15 joints
Links:
- removed link camera_visor
- added link camera_base_rgb
- added link camera_basenonrotated
- added link camera_holder; visual mesh filename=package://authoring/meshes/camera_holder_assem.STL
- added link camera_tripod
- added link panda_flange
Joints:
- removed joint camera_base_to_visor
- added joint camera_base_rgb_joint: type fixed, parent camera_base, child camera_base_rgb, origin xyz=0.0 -0.03 0.0 rpy=0.0 0.0 0.0
- added joint camera_holder_joint: type fixed, parent panda_flange, child camera_holder, origin xyz=0 0 0.0114808 rpy=3.14 0.0 0.0
- added joint camera_rotation: type fixed, parent camera_basenonrotated, child camera_tripod, origin xyz=0.0 0.0 0.0 rpy=0 -0.16069 0
- added joint camera_tripod_joint: type fixed, parent camera_tripod, child camera_base, origin xyz=0.062 0.0 0.0068 rpy=0 0 0
- added joint panda_flange_joint: type fixed, parent ft_sensor_link, child panda_flange, origin xyz=0 0 0.04 rpy=0 0 -0.785398163397
- joint fake_base: child camera_base -> camera_basenonrotated; origin xyz=0.029 -0.056 0.01 rpy=3.14 -1.57 -0.785 -> xyz=0.093997 0.0 0.0266868 rpy=3.14 -1.57 0.0; parent panda_link8 -> panda_flange

Commit message: Another small adjustment to camera height

File: src/authoring/urdfs/panda.urdf (robot description, URDF)
Before this commit: robot panda_kinect, 20 links, 19 joints
Joints:
- joint panda_flange_joint: origin xyz=0 0 0.04 rpy=0 0 -0.785398163397 -> xyz=0 0 0.043 rpy=0 0 -0.785398163397
