Commit message: Fixed package name

File: urdfs/panda.urdf (robot description, URDF)
Before this commit: robot panda_kinect, 20 links, 19 joints
Links:
- link camera_body: geometry visual mesh filename=package://panda-primitives/meshes/visual/kinect-model.stl
- link camera_holder: geometry visual mesh filename=package://panda-primitives/meshes/camera_holder_assem.STL
- link ft_sensor_link: geometry collision mesh filename=package://panda-primitives/meshes/force_torque_sensor.stl; visual mesh filename=package://panda-primitives/meshes/force_torque_sensor.dae
- link panda_hand: geometry collision mesh filename=package://panda-primitives/meshes/collision/hand.stl; visual mesh filename=package://panda-primitives/meshes/visual/hand.dae
- link panda_leftfinger: geometry collision mesh filename=package://panda-primitives/meshes/collision/finger.stl; visual mesh filename=package://panda-primitives/meshes/visual/finger.dae
- link panda_link0: geometry collision mesh filename=package://panda-primitives/meshes/collision/link0.stl; visual mesh filename=package://panda-primitives/meshes/visual/link0.dae
- link panda_link1: geometry collision mesh filename=package://panda-primitives/meshes/collision/link1.stl; visual mesh filename=package://panda-primitives/meshes/visual/link1.dae
- link panda_link2: geometry collision mesh filename=package://panda-primitives/meshes/collision/link2.stl; visual mesh filename=package://panda-primitives/meshes/visual/link2.dae
- link panda_link3: geometry collision mesh filename=package://panda-primitives/meshes/collision/link3.stl; visual mesh filename=package://panda-primitives/meshes/visual/link3.dae
- link panda_link4: geometry collision mesh filename=package://panda-primitives/meshes/collision/link4.stl; visual mesh filename=package://panda-primitives/meshes/visual/link4.dae
- link panda_link5: geometry collision mesh filename=package://panda-primitives/meshes/collision/link5.stl; visual mesh filename=package://panda-primitives/meshes/visual/link5.dae
- link panda_link6: geometry collision mesh filename=package://panda-primitives/meshes/collision/link6.stl; visual mesh filename=package://panda-primitives/meshes/visual/link6.dae
- link panda_link7: geometry collision mesh filename=package://panda-primitives/meshes/collision/link7.stl; visual mesh filename=package://panda-primitives/meshes/visual/link7.dae
- link panda_rightfinger: geometry collision mesh filename=package://panda-primitives/meshes/collision/finger.stl; visual mesh filename=package://panda-primitives/meshes/visual/finger.dae
